File: PCB_LeftPanel/I2C_Exp.sch (KiCad schematic (older format))
At the start: 4 parts, among them J32 DB9_Female, J33 DB9_Female, J34 DB9_Female, J35 DB9_Female

Commit message: Add files via upload
Parts:
- removed J33, J34, J35: DB9_Female, Connector_Dsub:DSUB-9_Female_Horizontal_P2.77x2.54mm_EdgePinOffset9.40mm, symbol Connector:DB9_Female
- J32: footprint Connector_Dsub:DSUB-9_Female_Horizontal_P2.77x2.54mm_EdgePinOffset9.40mm -> Connector_Dsub:DSUB-9_Female_Vertical_P2.77x2.84mm_MountingHoles
Connections:
- net GND: now also J32.2, J32.3; no longer J32.1, J32.5
- net SCL: now also J32.5; no longer J32.2
- net SDA: now also J32.1; no longer J32.3
