File: PCB_LeftPanel/InputOutputPins.sch (KiCad schematic (older format))
At the start: 190 parts, among them J10 HDR_2x8, J11 HDR_2x8, J12 HDR_2x8, J13 HDR_2x8, J14 HDR_2x8, J15 HDR_2x8, J16 HDR_2x8, J17 HDR_2x8, J18 HDR_2x8, J19 HDR_2x8, J20 HDR_2x8, J21 HDR_2x8, J22 HDR_2x8, J23 HDR_2x8, J4 HDR_2x8, J5 HDR_2x8, J6 HDR_2x8, J7 HDR_2x8, J8 HDR_2x8, J9 HDR_2x8, Q1 PNP, Q10 PNP, Q2 PNP, Q3 PNP, Q4 PNP, Q5 PNP, Q6 PNP, Q7 PNP, Q8 PNP, Q9 PNP

Commit message: Add files via upload
Parts:
- removed Q1, Q10, Q2, Q3, Q4, Q5, Q6, Q7, Q8, Q9: PNP, Transistor:2N4402, symbol Device:Q_PNP_BEC
- added U4, U5: 74AHC04, Package_DIP:DIP-14_W7.62mm, symbol 74xx:74AHC04
Connections:
- net labels added: GND
- wire segments 425 -> 413

Commit message: Add files via upload
Parts:
- J10, J11, J12, J13, J14, J15, J16, J17, J18, J19, J20, J21, J22, J23, J4, J5, J6, J7, J8, J9: symbol Connector_Generic:Conn_02x08_Row_Letter_First -> Connector_Generic:Conn_02x08_Odd_Even
Connections:
- net at R7.1: now also J4.1 (Pin_1); no longer J4.a1 (Pin_a1)
- net at R8.1: now also J4.3 (Pin_3); no longer J4.a2 (Pin_a2)
- net at R9.1: now also J4.5 (Pin_5); no longer J4.a3 (Pin_a3)
- net at R10.1: now also J4.7 (Pin_7); no longer J4.a4 (Pin_a4)
- net at R11.1: now also J4.9 (Pin_9); no longer J4.a5 (Pin_a5)
- net at R12.1: now also J4.11 (Pin_11); no longer J4.a6 (Pin_a6)
- net at R13.1: now also J4.13 (Pin_13); no longer J4.a7 (Pin_a7)
- net at R14.1: now also J4.15 (Pin_15); no longer J4.a8 (Pin_a8)
- net at D7.2 (A): now also J5.1 (Pin_1); no longer J5.a1 (Pin_a1)
- net at D8.2 (A): now also J5.3 (Pin_3); no longer J5.a2 (Pin_a2)
- net at D9.2 (A): now also J5.5 (Pin_5); no longer J5.a3 (Pin_a3)
- net at D10.2 (A): now also J5.7 (Pin_7); no longer J5.a4 (Pin_a4)
- net at D11.2 (A): now also J5.9 (Pin_9); no longer J5.a5 (Pin_a5)
- net at D12.2 (A): now also J5.11 (Pin_11); no longer J5.a6 (Pin_a6)
- net at D13.2 (A): now also J5.13 (Pin_13); no longer J5.a7 (Pin_a7)
- net at D14.2 (A): now also J5.15 (Pin_15); no longer J5.a8 (Pin_a8)
- net at R15.1: now also J6.1 (Pin_1); no longer J6.a1 (Pin_a1)
- net at R16.1: now also J6.3 (Pin_3); no longer J6.a2 (Pin_a2)
- net at R17.1: now also J6.5 (Pin_5); no longer J6.a3 (Pin_a3)
- net at R18.1: now also J6.7 (Pin_7); no longer J6.a4 (Pin_a4)
- net at R19.1: now also J6.9 (Pin_9); no longer J6.a5 (Pin_a5)
- net at R20.1: now also J6.11 (Pin_11); no longer J6.a6 (Pin_a6)
- net at R21.1: now also J6.13 (Pin_13); no longer J6.a7 (Pin_a7)
- net at R22.1: now also J6.15 (Pin_15); no longer J6.a8 (Pin_a8)
- net at D15.2 (A): now also J7.1 (Pin_1); no longer J7.a1 (Pin_a1)
- net at D16.2 (A): now also J7.3 (Pin_3); no longer J7.a2 (Pin_a2)
- net at D17.2 (A): now also J7.5 (Pin_5); no longer J7.a3 (Pin_a3)
- net at D18.2 (A): now also J7.7 (Pin_7); no longer J7.a4 (Pin_a4)
- net at D19.2 (A): now also J7.9 (Pin_9); no longer J7.a5 (Pin_a5)
- net at D20.2 (A): now also J7.11 (Pin_11); no longer J7.a6 (Pin_a6)
- net at D21.2 (A): now also J7.13 (Pin_13); no longer J7.a7 (Pin_a7)
- net at D22.2 (A): now also J7.15 (Pin_15); no longer J7.a8 (Pin_a8)
- net at R23.1: now also J8.1 (Pin_1); no longer J8.a1 (Pin_a1)
- net at R24.1: now also J8.3 (Pin_3); no longer J8.a2 (Pin_a2)
- net at R25.1: now also J8.5 (Pin_5); no longer J8.a3 (Pin_a3)
- net at R26.1: now also J8.7 (Pin_7); no longer J8.a4 (Pin_a4)
- net at R27.1: now also J8.9 (Pin_9); no longer J8.a5 (Pin_a5)
- net at R28.1: now also J8.11 (Pin_11); no longer J8.a6 (Pin_a6)
- net at R29.1: now also J8.13 (Pin_13); no longer J8.a7 (Pin_a7)
- net at R30.1: now also J8.15 (Pin_15); no longer J8.a8 (Pin_a8)
- net at D23.2 (A): now also J9.1 (Pin_1); no longer J9.a1 (Pin_a1)
- net at D24.2 (A): now also J9.3 (Pin_3); no longer J9.a2 (Pin_a2)
- net at D25.2 (A): now also J9.5 (Pin_5); no longer J9.a3 (Pin_a3)
- net at D26.2 (A): now also J9.7 (Pin_7); no longer J9.a4 (Pin_a4)
- net at D27.2 (A): now also J9.9 (Pin_9); no longer J9.a5 (Pin_a5)
- net at D28.2 (A): now also J9.11 (Pin_11); no longer J9.a6 (Pin_a6)
- net at D29.2 (A): now also J9.13 (Pin_13); no longer J9.a7 (Pin_a7)
- net at D30.2 (A): now also J9.15 (Pin_15); no longer J9.a8 (Pin_a8)
- net at R31.1: now also J10.1 (Pin_1); no longer J10.a1 (Pin_a1)
- net at R32.1: now also J10.3 (Pin_3); no longer J10.a2 (Pin_a2)
- net at R33.1: now also J10.5 (Pin_5); no longer J10.a3 (Pin_a3)
- net at R34.1: now also J10.7 (Pin_7); no longer J10.a4 (Pin_a4)
- net at R35.1: now also J10.9 (Pin_9); no longer J10.a5 (Pin_a5)
- net at R36.1: now also J10.11 (Pin_11); no longer J10.a6 (Pin_a6)
- net at R37.1: now also J10.13 (Pin_13); no longer J10.a7 (Pin_a7)
- net at R38.1: now also J10.15 (Pin_15); no longer J10.a8 (Pin_a8)
- net at D31.2 (A): now also J11.1 (Pin_1); no longer J11.a1 (Pin_a1)
- net at D32.2 (A): now also J11.3 (Pin_3); no longer J11.a2 (Pin_a2)
- net at D33.2 (A): now also J11.5 (Pin_5); no longer J11.a3 (Pin_a3)
- net at D34.2 (A): now also J11.7 (Pin_7); no longer J11.a4 (Pin_a4)
- net at D35.2 (A): now also J11.9 (Pin_9); no longer J11.a5 (Pin_a5)
- net at D36.2 (A): now also J11.11 (Pin_11); no longer J11.a6 (Pin_a6)
- net at D37.2 (A): now also J11.13 (Pin_13); no longer J11.a7 (Pin_a7)
- net at D38.2 (A): now also J11.15 (Pin_15); no longer J11.a8 (Pin_a8)
- net at R39.1: now also J12.1 (Pin_1); no longer J12.a1 (Pin_a1)
- net at R40.1: now also J12.3 (Pin_3); no longer J12.a2 (Pin_a2)
- net at R41.1: now also J12.5 (Pin_5); no longer J12.a3 (Pin_a3)
- net at R42.1: now also J12.7 (Pin_7); no longer J12.a4 (Pin_a4)
- net at R43.1: now also J12.9 (Pin_9); no longer J12.a5 (Pin_a5)
- net at R44.1: now also J12.11 (Pin_11); no longer J12.a6 (Pin_a6)
- net at R45.1: now also J12.13 (Pin_13); no longer J12.a7 (Pin_a7)
- net at R46.1: now also J12.15 (Pin_15); no longer J12.a8 (Pin_a8)
- net at D39.2 (A): now also J13.1 (Pin_1); no longer J13.a1 (Pin_a1)
- net at D40.2 (A): now also J13.3 (Pin_3); no longer J13.a2 (Pin_a2)
- net at D41.2 (A): now also J13.5 (Pin_5); no longer J13.a3 (Pin_a3)
- net at D42.2 (A): now also J13.7 (Pin_7); no longer J13.a4 (Pin_a4)
- net at D43.2 (A): now also J13.9 (Pin_9); no longer J13.a5 (Pin_a5)
- net at D44.2 (A): now also J13.11 (Pin_11); no longer J13.a6 (Pin_a6)
- net at D45.2 (A): now also J13.13 (Pin_13); no longer J13.a7 (Pin_a7)
- net at D46.2 (A): now also J13.15 (Pin_15); no longer J13.a8 (Pin_a8)
- net at R47.1: now also J14.1 (Pin_1); no longer J14.a1 (Pin_a1)
- net at R48.1: now also J14.3 (Pin_3); no longer J14.a2 (Pin_a2)
- net at R49.1: now also J14.5 (Pin_5); no longer J14.a3 (Pin_a3)
- net at R50.1: now also J14.7 (Pin_7); no longer J14.a4 (Pin_a4)
- net at R51.1: now also J14.9 (Pin_9); no longer J14.a5 (Pin_a5)
- net at R52.1: now also J14.11 (Pin_11); no longer J14.a6 (Pin_a6)
- net at R53.1: now also J14.13 (Pin_13); no longer J14.a7 (Pin_a7)
- net at R54.1: now also J14.15 (Pin_15); no longer J14.a8 (Pin_a8)
- net at D47.2 (A): now also J15.1 (Pin_1); no longer J15.a1 (Pin_a1)
- net at D48.2 (A): now also J15.3 (Pin_3); no longer J15.a2 (Pin_a2)
- net at D49.2 (A): now also J15.5 (Pin_5); no longer J15.a3 (Pin_a3)
- net at D50.2 (A): now also J15.7 (Pin_7); no longer J15.a4 (Pin_a4)
- net at D51.2 (A): now also J15.9 (Pin_9); no longer J15.a5 (Pin_a5)
- net at D52.2 (A): now also J15.11 (Pin_11); no longer J15.a6 (Pin_a6)
- net at D53.2 (A): now also J15.13 (Pin_13); no longer J15.a7 (Pin_a7)
- net at D54.2 (A): now also J15.15 (Pin_15); no longer J15.a8 (Pin_a8)
- net at R55.1: now also J16.1 (Pin_1); no longer J16.a1 (Pin_a1)
- net at R56.1: now also J16.3 (Pin_3); no longer J16.a2 (Pin_a2)
- net at R57.1: now also J16.5 (Pin_5); no longer J16.a3 (Pin_a3)
- net at R58.1: now also J16.7 (Pin_7); no longer J16.a4 (Pin_a4)
- net at R59.1: now also J16.9 (Pin_9); no longer J16.a5 (Pin_a5)
- net at R60.1: now also J16.11 (Pin_11); no longer J16.a6 (Pin_a6)
- net at R61.1: now also J16.13 (Pin_13); no longer J16.a7 (Pin_a7)
- net at R62.1: now also J16.15 (Pin_15); no longer J16.a8 (Pin_a8)
- net at D55.2 (A): now also J17.1 (Pin_1); no longer J17.a1 (Pin_a1)
- net at D56.2 (A): now also J17.3 (Pin_3); no longer J17.a2 (Pin_a2)
- net at D57.2 (A): now also J17.5 (Pin_5); no longer J17.a3 (Pin_a3)
- net at D58.2 (A): now also J17.7 (Pin_7); no longer J17.a4 (Pin_a4)
- net at D59.2 (A): now also J17.9 (Pin_9); no longer J17.a5 (Pin_a5)
- net at D60.2 (A): now also J17.11 (Pin_11); no longer J17.a6 (Pin_a6)
- net at D61.2 (A): now also J17.13 (Pin_13); no longer J17.a7 (Pin_a7)
- net at D62.2 (A): now also J17.15 (Pin_15); no longer J17.a8 (Pin_a8)
- net at R63.1: now also J18.1 (Pin_1); no longer J18.a1 (Pin_a1)
- net at R64.1: now also J18.3 (Pin_3); no longer J18.a2 (Pin_a2)
- net at R65.1: now also J18.5 (Pin_5); no longer J18.a3 (Pin_a3)
- net at R66.1: now also J18.7 (Pin_7); no longer J18.a4 (Pin_a4)
- net at R67.1: now also J18.9 (Pin_9); no longer J18.a5 (Pin_a5)
- net at R68.1: now also J18.11 (Pin_11); no longer J18.a6 (Pin_a6)
- net at R69.1: now also J18.13 (Pin_13); no longer J18.a7 (Pin_a7)
- net at R70.1: now also J18.15 (Pin_15); no longer J18.a8 (Pin_a8)
- net at D63.2 (A): now also J19.1 (Pin_1); no longer J19.a1 (Pin_a1)
- net at D64.2 (A): now also J19.3 (Pin_3); no longer J19.a2 (Pin_a2)
- net at D65.2 (A): now also J19.5 (Pin_5); no longer J19.a3 (Pin_a3)
- net at D66.2 (A): now also J19.7 (Pin_7); no longer J19.a4 (Pin_a4)
- net at D67.2 (A): now also J19.9 (Pin_9); no longer J19.a5 (Pin_a5)
- net at D68.2 (A): now also J19.11 (Pin_11); no longer J19.a6 (Pin_a6)
- net at D69.2 (A): now also J19.13 (Pin_13); no longer J19.a7 (Pin_a7)
- net at D70.2 (A): now also J19.15 (Pin_15); no longer J19.a8 (Pin_a8)
- net at R71.1: now also J20.1 (Pin_1); no longer J20.a1 (Pin_a1)
- net at R72.1: now also J20.3 (Pin_3); no longer J20.a2 (Pin_a2)
- net at R73.1: now also J20.5 (Pin_5); no longer J20.a3 (Pin_a3)
- net at R74.1: now also J20.7 (Pin_7); no longer J20.a4 (Pin_a4)
- net at R75.1: now also J20.9 (Pin_9); no longer J20.a5 (Pin_a5)
- net at R76.1: now also J20.11 (Pin_11); no longer J20.a6 (Pin_a6)
- net at R77.1: now also J20.13 (Pin_13); no longer J20.a7 (Pin_a7)
- net at R78.1: now also J20.15 (Pin_15); no longer J20.a8 (Pin_a8)
- net at D71.2 (A): now also J21.1 (Pin_1); no longer J21.a1 (Pin_a1)
- net at D72.2 (A): now also J21.3 (Pin_3); no longer J21.a2 (Pin_a2)
- net at D73.2 (A): now also J21.5 (Pin_5); no longer J21.a3 (Pin_a3)
- net at D74.2 (A): now also J21.7 (Pin_7); no longer J21.a4 (Pin_a4)
- net at D75.2 (A): now also J21.9 (Pin_9); no longer J21.a5 (Pin_a5)
- net at D76.2 (A): now also J21.11 (Pin_11); no longer J21.a6 (Pin_a6)
- net at D77.2 (A): now also J21.13 (Pin_13); no longer J21.a7 (Pin_a7)
- net at D78.2 (A): now also J21.15 (Pin_15); no longer J21.a8 (Pin_a8)
- net at R79.1: now also J22.1 (Pin_1); no longer J22.a1 (Pin_a1)
- net at R80.1: now also J22.3 (Pin_3); no longer J22.a2 (Pin_a2)
- net at R81.1: now also J22.5 (Pin_5); no longer J22.a3 (Pin_a3)
- net at R82.1: now also J22.7 (Pin_7); no longer J22.a4 (Pin_a4)
- net at R83.1: now also J22.9 (Pin_9); no longer J22.a5 (Pin_a5)
- net at R84.1: now also J22.11 (Pin_11); no longer J22.a6 (Pin_a6)
- net at R85.1: now also J22.13 (Pin_13); no longer J22.a7 (Pin_a7)
- net at R86.1: now also J22.15 (Pin_15); no longer J22.a8 (Pin_a8)
- net at D79.2 (A): now also J23.1 (Pin_1); no longer J23.a1 (Pin_a1)
- net at D80.2 (A): now also J23.3 (Pin_3); no longer J23.a2 (Pin_a2)
- net at D81.2 (A): now also J23.5 (Pin_5); no longer J23.a3 (Pin_a3)
- net at D82.2 (A): now also J23.7 (Pin_7); no longer J23.a4 (Pin_a4)
- net at D83.2 (A): now also J23.9 (Pin_9); no longer J23.a5 (Pin_a5)
- net at D84.2 (A): now also J23.11 (Pin_11); no longer J23.a6 (Pin_a6)
- net at D85.2 (A): now also J23.13 (Pin_13); no longer J23.a7 (Pin_a7)
- net at D86.2 (A): now also J23.15 (Pin_15); no longer J23.a8 (Pin_a8)
- new net: J4.10 (Pin_10), J4.12 (Pin_12), J4.14 (Pin_14), J4.16 (Pin_16), J4.2 (Pin_2), J4.4 (Pin_4), J4.6 (Pin_6), J4.8 (Pin_8), J5.10 (Pin_10), J5.12 (Pin_12), J5.14 (Pin_14), J5.16 (Pin_16), J5.2 (Pin_2), J5.4 (Pin_4), J5.6 (Pin_6), J5.8 (Pin_8), U4.2
- new net: J6.10 (Pin_10), J6.12 (Pin_12), J6.14 (Pin_14), J6.16 (Pin_16), J6.2 (Pin_2), J6.4 (Pin_4), J6.6 (Pin_6), J6.8 (Pin_8), J7.10 (Pin_10), J7.12 (Pin_12), J7.14 (Pin_14), J7.16 (Pin_16), J7.2 (Pin_2), J7.4 (Pin_4), J7.6 (Pin_6), J7.8 (Pin_8), U4.4
- new net: J8.10 (Pin_10), J8.12 (Pin_12), J8.14 (Pin_14), J8.16 (Pin_16), J8.2 (Pin_2), J8.4 (Pin_4), J8.6 (Pin_6), J8.8 (Pin_8), J9.10 (Pin_10), J9.12 (Pin_12), J9.14 (Pin_14), J9.16 (Pin_16), J9.2 (Pin_2), J9.4 (Pin_4), J9.6 (Pin_6), J9.8 (Pin_8), U4.6
- new net: J10.10 (Pin_10), J10.12 (Pin_12), J10.14 (Pin_14), J10.16 (Pin_16), J10.2 (Pin_2), J10.4 (Pin_4), J10.6 (Pin_6), J10.8 (Pin_8), J11.10 (Pin_10), J11.12 (Pin_12), J11.14 (Pin_14), J11.16 (Pin_16), J11.2 (Pin_2), J11.4 (Pin_4), J11.6 (Pin_6), J11.8 (Pin_8), U4.8
- new net: J12.10 (Pin_10), J12.12 (Pin_12), J12.14 (Pin_14), J12.16 (Pin_16), J12.2 (Pin_2), J12.4 (Pin_4), J12.6 (Pin_6), J12.8 (Pin_8), J13.10 (Pin_10), J13.12 (Pin_12), J13.14 (Pin_14), J13.16 (Pin_16), J13.2 (Pin_2), J13.4 (Pin_4), J13.6 (Pin_6), J13.8 (Pin_8), U4.10
- new net: J14.10 (Pin_10), J14.12 (Pin_12), J14.14 (Pin_14), J14.16 (Pin_16), J14.2 (Pin_2), J14.4 (Pin_4), J14.6 (Pin_6), J14.8 (Pin_8), J15.10 (Pin_10), J15.12 (Pin_12), J15.14 (Pin_14), J15.16 (Pin_16), J15.2 (Pin_2), J15.4 (Pin_4), J15.6 (Pin_6), J15.8 (Pin_8), U4.12
- new net: J16.10 (Pin_10), J16.12 (Pin_12), J16.14 (Pin_14), J16.16 (Pin_16), J16.2 (Pin_2), J16.4 (Pin_4), J16.6 (Pin_6), J16.8 (Pin_8), J17.10 (Pin_10), J17.12 (Pin_12), J17.14 (Pin_14), J17.16 (Pin_16), J17.2 (Pin_2), J17.4 (Pin_4), J17.6 (Pin_6), J17.8 (Pin_8), U5.2
- new net: J18.10 (Pin_10), J18.12 (Pin_12), J18.14 (Pin_14), J18.16 (Pin_16), J18.2 (Pin_2), J18.4 (Pin_4), J18.6 (Pin_6), J18.8 (Pin_8), J19.10 (Pin_10), J19.12 (Pin_12), J19.14 (Pin_14), J19.16 (Pin_16), J19.2 (Pin_2), J19.4 (Pin_4), J19.6 (Pin_6), J19.8 (Pin_8), U5.4
- new net: J20.10 (Pin_10), J20.12 (Pin_12), J20.14 (Pin_14), J20.16 (Pin_16), J20.2 (Pin_2), J20.4 (Pin_4), J20.6 (Pin_6), J20.8 (Pin_8), J21.10 (Pin_10), J21.12 (Pin_12), J21.14 (Pin_14), J21.16 (Pin_16), J21.2 (Pin_2), J21.4 (Pin_4), J21.6 (Pin_6), J21.8 (Pin_8), U5.6
- new net: J22.10 (Pin_10), J22.12 (Pin_12), J22.14 (Pin_14), J22.16 (Pin_16), J22.2 (Pin_2), J22.4 (Pin_4), J22.6 (Pin_6), J22.8 (Pin_8), J23.10 (Pin_10), J23.12 (Pin_12), J23.14 (Pin_14), J23.16 (Pin_16), J23.2 (Pin_2), J23.4 (Pin_4), J23.6 (Pin_6), J23.8 (Pin_8), U5.8
Changed lines of the file:
@@
 Q9
 $Comp
-L Connector_Generic:Conn_02x08_Row_Letter_First J4
+L Connector_Generic:Conn_02x08_Odd_Even J4
 U 1 1 612E77DB
 P 1850 2350
@@
 $EndComp
 $Comp
-L Connector_Generic:Conn_02x08_Row_Letter_First J5
+L Connector_Generic:Conn_02x08_Odd_Even J5
 U 1 1 612ECDC4
 P 1850 3400
@@
 PC7
 $Comp
-L Connector_Generic:Conn_02x08_Row_Letter_First J6
+L Connector_Generic:Conn_02x08_Odd_Even J6
 U 1 1 614108C8
 P 1850 4650
@@
 $EndComp
 $Comp
-L Connector_Generic:Conn_02x08_Row_Letter_First J7
+L Connector_Generic:Conn_02x08_Odd_Even J7
 U 1 1 61410BE6
 P 1850 5700
@@
 PC7
 $Comp
-L Connector_Generic:Conn_02x08_Row_Letter_First J8
+L Connector_Generic:Conn_02x08_Odd_Even J8
 U 1 1 6141BD97
 P 3800 2350
@@
 $EndComp
 $Comp
-L Connector_Generic:Conn_02x08_Row_Letter_First J9
+L Connector_Generic:Conn_02x08_Odd_Even J9
 U 1 1 6141C26D
 P 3800 3400
@@
 PC7
 $Comp
-L Connector_Generic:Conn_02x08_Row_Letter_First J10
+L Connector_Generic:Conn_02x08_Odd_Even J10
 U 1 1 6141C33F
 P 3800 4650
@@
 $EndComp
 $Comp
-L Connector_Generic:Conn_02x08_Row_Letter_First J11
+L Connector_Generic:Conn_02x08_Odd_Even J11
 U 1 1 6141C349
 P 3800 5700
@@
 PC7
 $Comp
-L Connector_Generic:Conn_02x08_Row_Letter_First J12
+L Connector_Generic:Conn_02x08_Odd_Even J12
 U 1 1 614CD134
 P 5800 2350
@@
 $EndComp
 $Comp
-L Connector_Generic:Conn_02x08_Row_Letter_First J13
+L Connector_Generic:Conn_02x08_Odd_Even J13
 U 1 1 614CD97A
 P 5800 3400
@@
 PC7
 $Comp
-L Connector_Generic:Conn_02x08_Row_Letter_First J14
+L Connector_Generic:Conn_02x08_Odd_Even J14
 U 1 1 614CDA4C
 P 5800 4650
@@
 $EndComp
 $Comp
-L Connector_Generic:Conn_02x08_Row_Letter_First J15
+L Connector_Generic:Conn_02x08_Odd_Even J15
 U 1 1 614CDA56
 P 5800 5700
@@
 PC7
 $Comp
-L Connector_Generic:Conn_02x08_Row_Letter_First J16
+L Connector_Generic:Conn_02x08_Odd_Even J16
 U 1 1 614CDB28
 P 7800 2350
@@
 $EndComp
 $Comp
-L Connector_Generic:Conn_02x08_Row_Letter_First J17
+L Connector_Generic:Conn_02x08_Odd_Even J17
 U 1 1 614CDB32
 P 7800 3400
@@
 PC7
 $Comp
-L Connector_Generic:Conn_02x08_Row_Letter_First J18
+L Connector_Generic:Conn_02x08_Odd_Even J18
 U 1 1 614CDC04
 P 7800 4650
@@
 $EndComp
 $Comp
-L Connector_Generic:Conn_02x08_Row_Letter_First J19
+L Connector_Generic:Conn_02x08_Odd_Even J19
 U 1 1 614CDC0E
 P 7800 5700
@@
 	6100 6000 6100 5900
 $Comp
-L Connector_Generic:Conn_02x08_Row_Letter_First J20
+L Connector_Generic:Conn_02x08_Odd_Even J20
 U 1 1 61622DE8
 P 9900 2350
@@
 $EndComp
 $Comp
-L Connector_Generic:Conn_02x08_Row_Letter_First J21
+L Connector_Generic:Conn_02x08_Odd_Even J21
 U 1 1 61622E3A
 P 9900 3400
@@
 PC7
 $Comp
-L Connector_Generic:Conn_02x08_Row_Letter_First J22
+L Connector_Generic:Conn_02x08_Odd_Even J22
 U 1 1 61622F0C
 P 9900 4650
@@
 $EndComp
 $Comp
-L Connector_Generic:Conn_02x08_Row_Letter_First J23
+L Connector_Generic:Conn_02x08_Odd_Even J23
 U 1 1 61622F16
 P 9900 5700

Commit message: Add files via upload
Update to Revision 4.A
Board now based on Arduino Leonardo / Uno
Parts:
- removed D13, D14, D21, D22, D29, D30, D37, D38, D45, D46, D53, D54, D61, D62, D69, D70, D77, D78, D85, D86: 1N4148, Diode_THT:D_DO-35_SOD27_P7.62mm_Horizontal, symbol Device:D_Small
- removed U4, U5: 74AHC04, Package_DIP:DIP-14_W7.62mm, symbol 74xx:74AHC04
Connections:
- net labels removed: +5V, GND, PC6, PC7
- wire segments 413 -> 376
