File: PCB_LeftPanel/PCB_LeftPanel.kicad_pcb (KiCad board)
At the start: 2 copper layers, 244 parts, among them J1 USB_B, J10 HDR_2x8, J11 HDR_2x8, J12 HDR_2x8, J13 HDR_2x8, J14 HDR_2x8, J15 HDR_2x8, J16 HDR_2x8, J17 HDR_2x8, J18 HDR_2x8, J19 HDR_2x8, J2 AVR-ISP-6, J20 HDR_2x8, J21 HDR_2x8, J22 HDR_2x8, J23 HDR_2x8, J24 Conn_01x03, J25 Conn_01x03, J26 Conn_01x03, J27 Conn_01x03, J28 Conn_01x03, J29 Conn_01x03, J3 Jack-DC, J30 Conn_01x03, J31 Conn_01x03, J32 DB9_Female, J33 DB9_Female, J34 DB9_Female, J35 DB9_Female, J4 HDR_2x8, J5 HDR_2x8, J6 HDR_2x8, J7 HDR_2x8, J8 HDR_2x8, J9 HDR_2x8, Q1 PNP, Q10 PNP, Q2 PNP, Q3 PNP, Q4 PNP, Q5 PNP, Q6 PNP, Q7 PNP, Q8 PNP, Q9 PNP, U1 ATmega16-16PU, U2 7442, U3 MCP2200-I-SO, Y1 Crystal

Commit message: Add files via upload
Parts:
- removed Q1, Q10, Q2, Q3, Q4, Q5, Q6, Q7, Q8, Q9: PNP, Transistor:2N4402
- added J36: Conn_01x08_Male, Connector_PinHeader_2.54mm:PinHeader_1x08_P2.54mm_Vertical, F.Cu at (113.0, 35.6)
- added U4: 74AHC04, Package_DIP:DIP-14_W7.62mm, F.Cu at (81.3, 113.0)
- added U5: 74AHC04, Package_DIP:DIP-14_W7.62mm, F.Cu at (109.2, 128.3)
- moved J32 265.5 mm to (343.5, 149.9)
- moved J35 265.5 mm to (495.9, 149.9)
- moved J33 265.5 mm to (394.3, 149.9)
- moved J34 265.5 mm to (445.1, 149.9)
- moved L3 87.4 mm to (120.7, 41.9)
- moved L1 87.1 mm to (120.7, 34.3)
- moved L2 75.7 mm to (120.7, 38.1)
- moved C11 57.8 mm to (43.8, -14.5)
- moved C13 57.8 mm to (53.6, -14.5)
- moved C16 57.8 mm to (63.3, -16.0)
- moved J24 57.8 mm to (80.9, -23.6)
- moved J26 57.8 mm to (86.6, -47.0)
- moved J27 57.8 mm to (122.2, -69.6)
- moved J30 57.8 mm to (76.3, -23.6)
- moved J31 57.8 mm to (94.1, -33.0)
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Routing:
- net +5V: track 195.7 -> 308.5 mm
- net GND: track 329.8 -> 284.6 mm
- net Q6: track 0.00 -> 34.9 mm
- net Q7: track 0.00 -> 31.1 mm
- net Q8: track 0.00 -> 25.4 mm
- net Q9: track 0.00 -> 20.7 mm
- net Q3: track 0.00 -> 20.1 mm
- net Q2: track 0.00 -> 17.6 mm
- net Q4: track 0.00 -> 14.9 mm
- net Q1: track 0.00 -> 12.5 mm
- net Q5: track 0.00 -> 9.94 mm
- net Q0: track 0.00 -> 8.02 mm

Commit message: Add files via upload
Parts:
- moved R71 376.5 mm to (69.2, 221.6), turned to 90 degrees
- moved R73 374.7 mm to (64.1, 221.6), turned to 90 degrees
- moved R3 371.6 mm to (48.9, 47.0), turned to 270 degrees
- moved R74 362.4 mm to (61.6, 221.6), turned to 90 degrees
- moved R78 356.9 mm to (51.4, 221.6), turned to 90 degrees
- moved R72 341.9 mm to (66.7, 221.6), turned to 90 degrees
- moved J35 334.9 mm to (162.6, 118.1), turned to 90 degrees
- moved D72 325.4 mm to (90.8, 214.0), turned to 270 degrees
- moved R79 322.0 mm to (117.5, 221.6), turned to 90 degrees
- moved D76 317.9 mm to (80.6, 214.0), turned to 270 degrees
- moved R70 315.4 mm to (99.7, 199.4), turned to 90 degrees
- moved R64 314.9 mm to (114.9, 199.4), turned to 90 degrees
- moved R76 313.7 mm to (56.5, 221.6), turned to 90 degrees
- moved D73 313.0 mm to (88.3, 214.0), turned to 270 degrees
- moved R68 308.7 mm to (104.8, 199.4), turned to 90 degrees
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Connections:
- C10 pad 1: GND -> /Analog Inputs/PA1
- C10 pad 2: /Analog Inputs/PA1 -> GND
- C11 pad 1: GND -> /Analog Inputs/PA2
- C11 pad 2: /Analog Inputs/PA2 -> GND
- C12 pad 1: GND -> /Analog Inputs/PA3
- C12 pad 2: /Analog Inputs/PA3 -> GND
- C13 pad 1: GND -> /Analog Inputs/PA4
- C13 pad 2: /Analog Inputs/PA4 -> GND
- C14 pad 1: GND -> /Analog Inputs/PA5
- C14 pad 2: /Analog Inputs/PA5 -> GND
- C15 pad 1: GND -> /Analog Inputs/PA6
- C15 pad 2: /Analog Inputs/PA6 -> GND
- C16 pad 1: GND -> /Analog Inputs/PA7
- C16 pad 2: /Analog Inputs/PA7 -> GND
- C3 pad 1: GND -> /Analog Inputs/PA0
- C3 pad 2: /Analog Inputs/PA0 -> GND
- J10 pad 1: (no net) -> Net-(J10-Pad1)
- J10 pad 10: (no net) -> Net-(J10-Pad10)
- J10 pad 11: (no net) -> Net-(J10-Pad11)
- J10 pad 12: (no net) -> Net-(J10-Pad10)
- J10 pad 13: (no net) -> Net-(J10-Pad13)
- J10 pad 14: (no net) -> Net-(J10-Pad10)
- J10 pad 15: (no net) -> Net-(J10-Pad15)
- J10 pad 16: (no net) -> Net-(J10-Pad10)
- J10 pad 2: (no net) -> Net-(J10-Pad10)
- J10 pad 3: (no net) -> Net-(J10-Pad3)
- J10 pad 4: (no net) -> Net-(J10-Pad10)
- J10 pad 5: (no net) -> Net-(J10-Pad5)
- J10 pad 6: (no net) -> Net-(J10-Pad10)
- J10 pad 7: (no net) -> Net-(J10-Pad7)
- J10 pad 8: (no net) -> Net-(J10-Pad10)
- J10 pad 9: (no net) -> Net-(J10-Pad9)
- J11 pad 1: (no net) -> Net-(D31-Pad2)
- J11 pad 10: (no net) -> Net-(J10-Pad10)
- J11 pad 11: (no net) -> Net-(D36-Pad2)
- J11 pad 12: (no net) -> Net-(J10-Pad10)
- J11 pad 13: (no net) -> Net-(D37-Pad2)
- J11 pad 14: (no net) -> Net-(J10-Pad10)
- J11 pad 15: (no net) -> Net-(D38-Pad2)
- J11 pad 16: (no net) -> Net-(J10-Pad10)
- J11 pad 2: (no net) -> Net-(J10-Pad10)
- J11 pad 3: (no net) -> Net-(D32-Pad2)
- J11 pad 4: (no net) -> Net-(J10-Pad10)
- J11 pad 5: (no net) -> Net-(D33-Pad2)
- J11 pad 6: (no net) -> Net-(J10-Pad10)
- J11 pad 7: (no net) -> Net-(D34-Pad2)
- J11 pad 8: (no net) -> Net-(J10-Pad10)
- J11 pad 9: (no net) -> Net-(D35-Pad2)
- J12 pad 1: (no net) -> Net-(J12-Pad1)
- J12 pad 10: (no net) -> Net-(J12-Pad10)
- J12 pad 11: (no net) -> Net-(J12-Pad11)
- J12 pad 12: (no net) -> Net-(J12-Pad10)
- J12 pad 13: (no net) -> Net-(J12-Pad13)
- J12 pad 14: (no net) -> Net-(J12-Pad10)
- J12 pad 15: (no net) -> Net-(J12-Pad15)
- J12 pad 16: (no net) -> Net-(J12-Pad10)
- J12 pad 2: (no net) -> Net-(J12-Pad10)
- J12 pad 3: (no net) -> Net-(J12-Pad3)
- J12 pad 4: (no net) -> Net-(J12-Pad10)
- J12 pad 5: (no net) -> Net-(J12-Pad5)
- J12 pad 6: (no net) -> Net-(J12-Pad10)
- J12 pad 7: (no net) -> Net-(J12-Pad7)
- J12 pad 8: (no net) -> Net-(J12-Pad10)
- J12 pad 9: (no net) -> Net-(J12-Pad9)
- J13 pad 1: (no net) -> Net-(D39-Pad2)
- J13 pad 10: (no net) -> Net-(J12-Pad10)
- J13 pad 11: (no net) -> Net-(D44-Pad2)
- J13 pad 12: (no net) -> Net-(J12-Pad10)
- J13 pad 13: (no net) -> Net-(D45-Pad2)
- J13 pad 14: (no net) -> Net-(J12-Pad10)
- J13 pad 15: (no net) -> Net-(D46-Pad2)
- J13 pad 16: (no net) -> Net-(J12-Pad10)
- J13 pad 2: (no net) -> Net-(J12-Pad10)
- J13 pad 3: (no net) -> Net-(D40-Pad2)
- J13 pad 4: (no net) -> Net-(J12-Pad10)
- J13 pad 5: (no net) -> Net-(D41-Pad2)
- J13 pad 6: (no net) -> Net-(J12-Pad10)
- J13 pad 7: (no net) -> Net-(D42-Pad2)
- J13 pad 8: (no net) -> Net-(J12-Pad10)
- J13 pad 9: (no net) -> Net-(D43-Pad2)
- J14 pad 1: (no net) -> Net-(J14-Pad1)
- J14 pad 10: (no net) -> Net-(J14-Pad10)
- J14 pad 11: (no net) -> Net-(J14-Pad11)
- J14 pad 12: (no net) -> Net-(J14-Pad10)
- J14 pad 13: (no net) -> Net-(J14-Pad13)
- J14 pad 14: (no net) -> Net-(J14-Pad10)
- J14 pad 15: (no net) -> Net-(J14-Pad15)
- J14 pad 16: (no net) -> Net-(J14-Pad10)
- J14 pad 2: (no net) -> Net-(J14-Pad10)
- J14 pad 3: (no net) -> Net-(J14-Pad3)
- J14 pad 4: (no net) -> Net-(J14-Pad10)
- J14 pad 5: (no net) -> Net-(J14-Pad5)
- J14 pad 6: (no net) -> Net-(J14-Pad10)
- J14 pad 7: (no net) -> Net-(J14-Pad7)
- J14 pad 8: (no net) -> Net-(J14-Pad10)
- J14 pad 9: (no net) -> Net-(J14-Pad9)
- J15 pad 1: (no net) -> Net-(D47-Pad2)
- J15 pad 10: (no net) -> Net-(J14-Pad10)
- J15 pad 11: (no net) -> Net-(D52-Pad2)
- J15 pad 12: (no net) -> Net-(J14-Pad10)
- J15 pad 13: (no net) -> Net-(D53-Pad2)
- J15 pad 14: (no net) -> Net-(J14-Pad10)
- J15 pad 15: (no net) -> Net-(D54-Pad2)
- J15 pad 16: (no net) -> Net-(J14-Pad10)
- J15 pad 2: (no net) -> Net-(J14-Pad10)
- J15 pad 3: (no net) -> Net-(D48-Pad2)
- J15 pad 4: (no net) -> Net-(J14-Pad10)
- J15 pad 5: (no net) -> Net-(D49-Pad2)
- J15 pad 6: (no net) -> Net-(J14-Pad10)
- J15 pad 7: (no net) -> Net-(D50-Pad2)
- J15 pad 8: (no net) -> Net-(J14-Pad10)
- J15 pad 9: (no net) -> Net-(D51-Pad2)
- J16 pad 1: (no net) -> Net-(J16-Pad1)
- J16 pad 10: (no net) -> Net-(J16-Pad10)
- J16 pad 11: (no net) -> Net-(J16-Pad11)
- J16 pad 12: (no net) -> Net-(J16-Pad10)
- J16 pad 13: (no net) -> Net-(J16-Pad13)
- J16 pad 14: (no net) -> Net-(J16-Pad10)
- J16 pad 15: (no net) -> Net-(J16-Pad15)
- J16 pad 16: (no net) -> Net-(J16-Pad10)
- J16 pad 2: (no net) -> Net-(J16-Pad10)
- J16 pad 3: (no net) -> Net-(J16-Pad3)
- J16 pad 4: (no net) -> Net-(J16-Pad10)
- J16 pad 5: (no net) -> Net-(J16-Pad5)
- J16 pad 6: (no net) -> Net-(J16-Pad10)
- J16 pad 7: (no net) -> Net-(J16-Pad7)
- J16 pad 8: (no net) -> Net-(J16-Pad10)
- J16 pad 9: (no net) -> Net-(J16-Pad9)
- J17 pad 1: (no net) -> Net-(D55-Pad2)
- J17 pad 10: (no net) -> Net-(J16-Pad10)
- J17 pad 11: (no net) -> Net-(D60-Pad2)
- J17 pad 12: (no net) -> Net-(J16-Pad10)
- J17 pad 13: (no net) -> Net-(D61-Pad2)
- J17 pad 14: (no net) -> Net-(J16-Pad10)
- J17 pad 15: (no net) -> Net-(D62-Pad2)
- J17 pad 16: (no net) -> Net-(J16-Pad10)
- J17 pad 2: (no net) -> Net-(J16-Pad10)
- J17 pad 3: (no net) -> Net-(D56-Pad2)
- J17 pad 4: (no net) -> Net-(J16-Pad10)
- J17 pad 5: (no net) -> Net-(D57-Pad2)
- J17 pad 6: (no net) -> Net-(J16-Pad10)
- J17 pad 7: (no net) -> Net-(D58-Pad2)
- J17 pad 8: (no net) -> Net-(J16-Pad10)
- J17 pad 9: (no net) -> Net-(D59-Pad2)
- J18 pad 1: (no net) -> Net-(J18-Pad1)
- J18 pad 10: (no net) -> Net-(J18-Pad10)
- J18 pad 11: (no net) -> Net-(J18-Pad11)
- J18 pad 12: (no net) -> Net-(J18-Pad10)
- J18 pad 13: (no net) -> Net-(J18-Pad13)
- J18 pad 14: (no net) -> Net-(J18-Pad10)
- J18 pad 15: (no net) -> Net-(J18-Pad15)
- J18 pad 16: (no net) -> Net-(J18-Pad10)
- J18 pad 2: (no net) -> Net-(J18-Pad10)
- J18 pad 3: (no net) -> Net-(J18-Pad3)
- J18 pad 4: (no net) -> Net-(J18-Pad10)
- J18 pad 5: (no net) -> Net-(J18-Pad5)
- J18 pad 6: (no net) -> Net-(J18-Pad10)
- J18 pad 7: (no net) -> Net-(J18-Pad7)
- J18 pad 8: (no net) -> Net-(J18-Pad10)
- J18 pad 9: (no net) -> Net-(J18-Pad9)
- J19 pad 1: (no net) -> Net-(D63-Pad2)
- J19 pad 10: (no net) -> Net-(J18-Pad10)
- J19 pad 11: (no net) -> Net-(D68-Pad2)
- J19 pad 12: (no net) -> Net-(J18-Pad10)
- J19 pad 13: (no net) -> Net-(D69-Pad2)
- J19 pad 14: (no net) -> Net-(J18-Pad10)
- J19 pad 15: (no net) -> Net-(D70-Pad2)
- J19 pad 16: (no net) -> Net-(J18-Pad10)
- J19 pad 2: (no net) -> Net-(J18-Pad10)
- J19 pad 3: (no net) -> Net-(D64-Pad2)
- J19 pad 4: (no net) -> Net-(J18-Pad10)
- J19 pad 5: (no net) -> Net-(D65-Pad2)
- J19 pad 6: (no net) -> Net-(J18-Pad10)
- J19 pad 7: (no net) -> Net-(D66-Pad2)
- J19 pad 8: (no net) -> Net-(J18-Pad10)
- J19 pad 9: (no net) -> Net-(D67-Pad2)
- J20 pad 1: (no net) -> Net-(J20-Pad1)
- J20 pad 10: (no net) -> Net-(J20-Pad10)
- J20 pad 11: (no net) -> Net-(J20-Pad11)
- J20 pad 12: (no net) -> Net-(J20-Pad10)
- J20 pad 13: (no net) -> Net-(J20-Pad13)
- J20 pad 14: (no net) -> Net-(J20-Pad10)
- J20 pad 15: (no net) -> Net-(J20-Pad15)
- J20 pad 16: (no net) -> Net-(J20-Pad10)
- J20 pad 2: (no net) -> Net-(J20-Pad10)
- J20 pad 3: (no net) -> Net-(J20-Pad3)
- J20 pad 4: (no net) -> Net-(J20-Pad10)
- J20 pad 5: (no net) -> Net-(J20-Pad5)
- J20 pad 6: (no net) -> Net-(J20-Pad10)
- J20 pad 7: (no net) -> Net-(J20-Pad7)
- J20 pad 8: (no net) -> Net-(J20-Pad10)
- J20 pad 9: (no net) -> Net-(J20-Pad9)
- J21 pad 1: (no net) -> Net-(D71-Pad2)
- J21 pad 10: (no net) -> Net-(J20-Pad10)
- J21 pad 11: (no net) -> Net-(D76-Pad2)
- J21 pad 12: (no net) -> Net-(J20-Pad10)
- J21 pad 13: (no net) -> Net-(D77-Pad2)
- J21 pad 14: (no net) -> Net-(J20-Pad10)
- J21 pad 15: (no net) -> Net-(D78-Pad2)
- J21 pad 16: (no net) -> Net-(J20-Pad10)
- J21 pad 2: (no net) -> Net-(J20-Pad10)
- J21 pad 3: (no net) -> Net-(D72-Pad2)
- J21 pad 4: (no net) -> Net-(J20-Pad10)
- J21 pad 5: (no net) -> Net-(D73-Pad2)
- J21 pad 6: (no net) -> Net-(J20-Pad10)
- J21 pad 7: (no net) -> Net-(D74-Pad2)
- J21 pad 8: (no net) -> Net-(J20-Pad10)
- J21 pad 9: (no net) -> Net-(D75-Pad2)
- J22 pad 1: (no net) -> Net-(J22-Pad1)
- J22 pad 10: (no net) -> Net-(J22-Pad10)
- J22 pad 11: (no net) -> Net-(J22-Pad11)
- J22 pad 12: (no net) -> Net-(J22-Pad10)
- J22 pad 13: (no net) -> Net-(J22-Pad13)
- J22 pad 14: (no net) -> Net-(J22-Pad10)
- J22 pad 15: (no net) -> Net-(J22-Pad15)
- J22 pad 16: (no net) -> Net-(J22-Pad10)
- J22 pad 2: (no net) -> Net-(J22-Pad10)
- J22 pad 3: (no net) -> Net-(J22-Pad3)
- J22 pad 4: (no net) -> Net-(J22-Pad10)
- J22 pad 5: (no net) -> Net-(J22-Pad5)
- J22 pad 6: (no net) -> Net-(J22-Pad10)
- J22 pad 7: (no net) -> Net-(J22-Pad7)
- J22 pad 8: (no net) -> Net-(J22-Pad10)
- J22 pad 9: (no net) -> Net-(J22-Pad9)
- J23 pad 1: (no net) -> Net-(D79-Pad2)
- J23 pad 10: (no net) -> Net-(J22-Pad10)
- J23 pad 11: (no net) -> Net-(D84-Pad2)
- J23 pad 12: (no net) -> Net-(J22-Pad10)
- J23 pad 13: (no net) -> Net-(D85-Pad2)
- J23 pad 14: (no net) -> Net-(J22-Pad10)
- J23 pad 15: (no net) -> Net-(D86-Pad2)
- J23 pad 16: (no net) -> Net-(J22-Pad10)
- J23 pad 2: (no net) -> Net-(J22-Pad10)
- J23 pad 3: (no net) -> Net-(D80-Pad2)
- J23 pad 4: (no net) -> Net-(J22-Pad10)
- J23 pad 5: (no net) -> Net-(D81-Pad2)
- J23 pad 6: (no net) -> Net-(J22-Pad10)
- J23 pad 7: (no net) -> Net-(D82-Pad2)
- J23 pad 8: (no net) -> Net-(J22-Pad10)
- J23 pad 9: (no net) -> Net-(D83-Pad2)
- J4 pad 1: (no net) -> Net-(J4-Pad1)
- J4 pad 10: (no net) -> Net-(J4-Pad10)
- J4 pad 11: (no net) -> Net-(J4-Pad11)
- J4 pad 12: (no net) -> Net-(J4-Pad10)
- J4 pad 13: (no net) -> Net-(J4-Pad13)
- J4 pad 14: (no net) -> Net-(J4-Pad10)
- J4 pad 15: (no net) -> Net-(J4-Pad15)
- J4 pad 16: (no net) -> Net-(J4-Pad10)
- J4 pad 2: (no net) -> Net-(J4-Pad10)
- J4 pad 3: (no net) -> Net-(J4-Pad3)
- J4 pad 4: (no net) -> Net-(J4-Pad10)
- J4 pad 5: (no net) -> Net-(J4-Pad5)
- J4 pad 6: (no net) -> Net-(J4-Pad10)
- J4 pad 7: (no net) -> Net-(J4-Pad7)
- J4 pad 8: (no net) -> Net-(J4-Pad10)
- J4 pad 9: (no net) -> Net-(J4-Pad9)
- J5 pad 1: (no net) -> Net-(D7-Pad2)
- J5 pad 10: (no net) -> Net-(J4-Pad10)
- J5 pad 11: (no net) -> Net-(D12-Pad2)
- J5 pad 12: (no net) -> Net-(J4-Pad10)
- J5 pad 13: (no net) -> Net-(D13-Pad2)
- J5 pad 14: (no net) -> Net-(J4-Pad10)
- J5 pad 15: (no net) -> Net-(D14-Pad2)
- J5 pad 16: (no net) -> Net-(J4-Pad10)
- J5 pad 2: (no net) -> Net-(J4-Pad10)
- J5 pad 3: (no net) -> Net-(D8-Pad2)
- J5 pad 4: (no net) -> Net-(J4-Pad10)
- J5 pad 5: (no net) -> Net-(D9-Pad2)
- J5 pad 6: (no net) -> Net-(J4-Pad10)
- J5 pad 7: (no net) -> Net-(D10-Pad2)
- J5 pad 8: (no net) -> Net-(J4-Pad10)
- J5 pad 9: (no net) -> Net-(D11-Pad2)
- J6 pad 1: (no net) -> Net-(J6-Pad1)
- J6 pad 10: (no net) -> Net-(J6-Pad10)
- J6 pad 11: (no net) -> Net-(J6-Pad11)
- J6 pad 12: (no net) -> Net-(J6-Pad10)
- J6 pad 13: (no net) -> Net-(J6-Pad13)
- J6 pad 14: (no net) -> Net-(J6-Pad10)
- J6 pad 15: (no net) -> Net-(J6-Pad15)
- J6 pad 16: (no net) -> Net-(J6-Pad10)
- J6 pad 2: (no net) -> Net-(J6-Pad10)
- J6 pad 3: (no net) -> Net-(J6-Pad3)
- J6 pad 4: (no net) -> Net-(J6-Pad10)
- J6 pad 5: (no net) -> Net-(J6-Pad5)
- J6 pad 6: (no net) -> Net-(J6-Pad10)
- J6 pad 7: (no net) -> Net-(J6-Pad7)
- J6 pad 8: (no net) -> Net-(J6-Pad10)
- J6 pad 9: (no net) -> Net-(J6-Pad9)
- J7 pad 1: (no net) -> Net-(D15-Pad2)
- J7 pad 10: (no net) -> Net-(J6-Pad10)
- J7 pad 11: (no net) -> Net-(D20-Pad2)
- J7 pad 12: (no net) -> Net-(J6-Pad10)
- J7 pad 13: (no net) -> Net-(D21-Pad2)
- J7 pad 14: (no net) -> Net-(J6-Pad10)
- J7 pad 15: (no net) -> Net-(D22-Pad2)
- J7 pad 16: (no net) -> Net-(J6-Pad10)
- J7 pad 2: (no net) -> Net-(J6-Pad10)
- J7 pad 3: (no net) -> Net-(D16-Pad2)
- J7 pad 4: (no net) -> Net-(J6-Pad10)
- J7 pad 5: (no net) -> Net-(D17-Pad2)
- J7 pad 6: (no net) -> Net-(J6-Pad10)
- J7 pad 7: (no net) -> Net-(D18-Pad2)
- J7 pad 8: (no net) -> Net-(J6-Pad10)
- J7 pad 9: (no net) -> Net-(D19-Pad2)
- J8 pad 1: (no net) -> Net-(J8-Pad1)
- J8 pad 10: (no net) -> Net-(J8-Pad10)
- J8 pad 11: (no net) -> Net-(J8-Pad11)
- J8 pad 12: (no net) -> Net-(J8-Pad10)
- J8 pad 13: (no net) -> Net-(J8-Pad13)
- J8 pad 14: (no net) -> Net-(J8-Pad10)
- J8 pad 15: (no net) -> Net-(J8-Pad15)
- J8 pad 16: (no net) -> Net-(J8-Pad10)
- J8 pad 2: (no net) -> Net-(J8-Pad10)
- J8 pad 3: (no net) -> Net-(J8-Pad3)
- J8 pad 4: (no net) -> Net-(J8-Pad10)
- J8 pad 5: (no net) -> Net-(J8-Pad5)
- J8 pad 6: (no net) -> Net-(J8-Pad10)
- J8 pad 7: (no net) -> Net-(J8-Pad7)
- J8 pad 8: (no net) -> Net-(J8-Pad10)
- J8 pad 9: (no net) -> Net-(J8-Pad9)
- J9 pad 1: (no net) -> Net-(D23-Pad2)
- J9 pad 10: (no net) -> Net-(J8-Pad10)
- J9 pad 11: (no net) -> Net-(D28-Pad2)
- J9 pad 12: (no net) -> Net-(J8-Pad10)
- J9 pad 13: (no net) -> Net-(D29-Pad2)
- J9 pad 14: (no net) -> Net-(J8-Pad10)
- J9 pad 15: (no net) -> Net-(D30-Pad2)
- J9 pad 16: (no net) -> Net-(J8-Pad10)
- J9 pad 2: (no net) -> Net-(J8-Pad10)
- J9 pad 3: (no net) -> Net-(D24-Pad2)
- J9 pad 4: (no net) -> Net-(J8-Pad10)
- J9 pad 5: (no net) -> Net-(D25-Pad2)
- J9 pad 6: (no net) -> Net-(J8-Pad10)
- J9 pad 7: (no net) -> Net-(D26-Pad2)
- J9 pad 8: (no net) -> Net-(J8-Pad10)
- J9 pad 9: (no net) -> Net-(D27-Pad2)
- R10 pad 1: Net-(J4-Pada4) -> Net-(J4-Pad7)
- R11 pad 1: Net-(J4-Pada5) -> Net-(J4-Pad9)
- R12 pad 1: Net-(J4-Pada6) -> Net-(J4-Pad11)
- R13 pad 1: Net-(J4-Pada7) -> Net-(J4-Pad13)
- R14 pad 1: Net-(J4-Pada8) -> Net-(J4-Pad15)
- R15 pad 1: Net-(J6-Pada1) -> Net-(J6-Pad1)
- R16 pad 1: Net-(J6-Pada2) -> Net-(J6-Pad3)
- R17 pad 1: Net-(J6-Pada3) -> Net-(J6-Pad5)
- R18 pad 1: Net-(J6-Pada4) -> Net-(J6-Pad7)
- R19 pad 1: Net-(J6-Pada5) -> Net-(J6-Pad9)
- R20 pad 1: Net-(J6-Pada6) -> Net-(J6-Pad11)
- R21 pad 1: Net-(J6-Pada7) -> Net-(J6-Pad13)
- R22 pad 1: Net-(J6-Pada8) -> Net-(J6-Pad15)
- R23 pad 1: Net-(J8-Pada1) -> Net-(J8-Pad1)
- R24 pad 1: Net-(J8-Pada2) -> Net-(J8-Pad3)
- R25 pad 1: Net-(J8-Pada3) -> Net-(J8-Pad5)
- R26 pad 1: Net-(J8-Pada4) -> Net-(J8-Pad7)
- R27 pad 1: Net-(J8-Pada5) -> Net-(J8-Pad9)
- R28 pad 1: Net-(J8-Pada6) -> Net-(J8-Pad11)
- R29 pad 1: Net-(J8-Pada7) -> Net-(J8-Pad13)
- R30 pad 1: Net-(J8-Pada8) -> Net-(J8-Pad15)
- R31 pad 1: Net-(J10-Pada1) -> Net-(J10-Pad1)
- R32 pad 1: Net-(J10-Pada2) -> Net-(J10-Pad3)
- R33 pad 1: Net-(J10-Pada3) -> Net-(J10-Pad5)
- R34 pad 1: Net-(J10-Pada4) -> Net-(J10-Pad7)
- R35 pad 1: Net-(J10-Pada5) -> Net-(J10-Pad9)
- R36 pad 1: Net-(J10-Pada6) -> Net-(J10-Pad11)
- R37 pad 1: Net-(J10-Pada7) -> Net-(J10-Pad13)
- R38 pad 1: Net-(J10-Pada8) -> Net-(J10-Pad15)
- R39 pad 1: Net-(J12-Pada1) -> Net-(J12-Pad1)
- R40 pad 1: Net-(J12-Pada2) -> Net-(J12-Pad3)
- R41 pad 1: Net-(J12-Pada3) -> Net-(J12-Pad5)
- R42 pad 1: Net-(J12-Pada4) -> Net-(J12-Pad7)
- R43 pad 1: Net-(J12-Pada5) -> Net-(J12-Pad9)
- R44 pad 1: Net-(J12-Pada6) -> Net-(J12-Pad11)
- R45 pad 1: Net-(J12-Pada7) -> Net-(J12-Pad13)
- R46 pad 1: Net-(J12-Pada8) -> Net-(J12-Pad15)
- R47 pad 1: Net-(J14-Pada1) -> Net-(J14-Pad1)
- R48 pad 1: Net-(J14-Pada2) -> Net-(J14-Pad3)
- R49 pad 1: Net-(J14-Pada3) -> Net-(J14-Pad5)
- R50 pad 1: Net-(J14-Pada4) -> Net-(J14-Pad7)
- R51 pad 1: Net-(J14-Pada5) -> Net-(J14-Pad9)
- R52 pad 1: Net-(J14-Pada6) -> Net-(J14-Pad11)
- R53 pad 1: Net-(J14-Pada7) -> Net-(J14-Pad13)
- R54 pad 1: Net-(J14-Pada8) -> Net-(J14-Pad15)
- R55 pad 1: Net-(J16-Pada1) -> Net-(J16-Pad1)
- R56 pad 1: Net-(J16-Pada2) -> Net-(J16-Pad3)
- R57 pad 1: Net-(J16-Pada3) -> Net-(J16-Pad5)
- R58 pad 1: Net-(J16-Pada4) -> Net-(J16-Pad7)
- R59 pad 1: Net-(J16-Pada5) -> Net-(J16-Pad9)
- R60 pad 1: Net-(J16-Pada6) -> Net-(J16-Pad11)
- R61 pad 1: Net-(J16-Pada7) -> Net-(J16-Pad13)
- R62 pad 1: Net-(J16-Pada8) -> Net-(J16-Pad15)
- R63 pad 1: Net-(J18-Pada1) -> Net-(J18-Pad1)
- R64 pad 1: Net-(J18-Pada2) -> Net-(J18-Pad3)
- R65 pad 1: Net-(J18-Pada3) -> Net-(J18-Pad5)
- R66 pad 1: Net-(J18-Pada4) -> Net-(J18-Pad7)
- R67 pad 1: Net-(J18-Pada5) -> Net-(J18-Pad9)
- R68 pad 1: Net-(J18-Pada6) -> Net-(J18-Pad11)
- R69 pad 1: Net-(J18-Pada7) -> Net-(J18-Pad13)
- R7 pad 1: Net-(J4-Pada1) -> Net-(J4-Pad1)
- R70 pad 1: Net-(J18-Pada8) -> Net-(J18-Pad15)
- R71 pad 1: Net-(J20-Pada1) -> Net-(J20-Pad1)
- R72 pad 1: Net-(J20-Pada2) -> Net-(J20-Pad3)
- R73 pad 1: Net-(J20-Pada3) -> Net-(J20-Pad5)
- R74 pad 1: Net-(J20-Pada4) -> Net-(J20-Pad7)
- R75 pad 1: Net-(J20-Pada5) -> Net-(J20-Pad9)
- R76 pad 1: Net-(J20-Pada6) -> Net-(J20-Pad11)
- R77 pad 1: Net-(J20-Pada7) -> Net-(J20-Pad13)
- R78 pad 1: Net-(J20-Pada8) -> Net-(J20-Pad15)
- R79 pad 1: Net-(J22-Pada1) -> Net-(J22-Pad1)
- R8 pad 1: Net-(J4-Pada2) -> Net-(J4-Pad3)
- R80 pad 1: Net-(J22-Pada2) -> Net-(J22-Pad3)
- R81 pad 1: Net-(J22-Pada3) -> Net-(J22-Pad5)
- R82 pad 1: Net-(J22-Pada4) -> Net-(J22-Pad7)
- R83 pad 1: Net-(J22-Pada5) -> Net-(J22-Pad9)
- R84 pad 1: Net-(J22-Pada6) -> Net-(J22-Pad11)
- R85 pad 1: Net-(J22-Pada7) -> Net-(J22-Pad13)
- R86 pad 1: Net-(J22-Pada8) -> Net-(J22-Pad15)
- R9 pad 1: Net-(J4-Pada3) -> Net-(J4-Pad5)
- U4 pad 10: Net-(J12-Padb1) -> Net-(J12-Pad10)
- U4 pad 12: Net-(J14-Padb1) -> Net-(J14-Pad10)
- U4 pad 2: Net-(J4-Padb1) -> Net-(J4-Pad10)
- U4 pad 4: Net-(J6-Padb1) -> Net-(J6-Pad10)
- U4 pad 6: Net-(J8-Padb1) -> Net-(J8-Pad10)
- U4 pad 8: Net-(J10-Padb1) -> Net-(J10-Pad10)
- U5 pad 2: Net-(J16-Padb1) -> Net-(J16-Pad10)
- U5 pad 4: Net-(J18-Padb1) -> Net-(J18-Pad10)
- U5 pad 6: Net-(J20-Padb1) -> Net-(J20-Pad10)
- U5 pad 8: Net-(J22-Padb1) -> Net-(J22-Pad10)
Routing:
- net GND: track 284.6 -> 471.4 mm
- net +5V: track 308.5 -> 462.3 mm
- net /InputOutputPins/PB0: track 0.00 -> 139.5 mm
- net /InputOutputPins/PB1: track 0.00 -> 138.0 mm
- net /InputOutputPins/PB2: track 0.00 -> 135.1 mm
- net /InputOutputPins/PB3: track 0.00 -> 132.7 mm
- net /InputOutputPins/PB4: track 0.00 -> 130.3 mm
- net /InputOutputPins/PB5: track 31.4 -> 159.0 mm
- net /InputOutputPins/PB6: track 31.0 -> 155.9 mm
- net /InputOutputPins/PB7: track 34.6 -> 157.1 mm
- net /InputOutputPins/PC1: track 0.00 -> 95.7 mm
- net /InputOutputPins/PC0: track 0.00 -> 95.3 mm
- net /InputOutputPins/PC2: track 0.00 -> 94.8 mm
- net /InputOutputPins/PC7: track 0.00 -> 94.7 mm
- net /InputOutputPins/PC3: track 0.00 -> 94.7 mm
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
Commit message: Add files via upload
Parts:
- removed J33, J34, J35: DB9_Female, Connector_Dsub:DSUB-9_Female_Horizontal_P2.77x2.54mm_EdgePinOffset9.40mm
- J32: footprint Connector_Dsub:DSUB-9_Female_Horizontal_P2.77x2.54mm_EdgePinOffset9.40mm -> Connector_Dsub:DSUB-9_Female_Vertical_P2.77x2.84mm_MountingHoles
- moved J32 148.8 mm to (123.2, 74.9)
Connections:
- J32 pad 1: GND -> /InputOutputPins/PC1
- J32 pad 2: /InputOutputPins/PC0 -> GND
- J32 pad 3: /InputOutputPins/PC1 -> GND
- J32 pad 5: GND -> /InputOutputPins/PC0
Routing:
- net GND: track 471.4 -> 768.8 mm
- net Net-(J22-Pad10): track 0.00 -> 238.4 mm
- net /InputOutputPins/PB2: track 135.1 -> 361.9 mm, vias 0 -> 1
- net /InputOutputPins/PC7: track 94.7 -> 315.6 mm, vias 0 -> 1
- net Net-(J18-Pad10): track 0.00 -> 220.0 mm, vias 0 -> 2
- net /InputOutputPins/PC1: track 95.7 -> 313.7 mm, vias 0 -> 1
- net /InputOutputPins/PC6: track 94.7 -> 312.5 mm, vias 0 -> 1
- net /InputOutputPins/PC0: track 95.3 -> 313.0 mm, vias 0 -> 1
- net /InputOutputPins/PC5: track 94.7 -> 310.0 mm, vias 0 -> 1
- net /InputOutputPins/PB7: track 157.1 -> 369.1 mm, vias 0 -> 1
- net /InputOutputPins/PC4: track 94.7 -> 306.2 mm, vias 0 -> 1
- net /InputOutputPins/PB6: track 155.9 -> 366.8 mm, vias 0 -> 1
- net /InputOutputPins/PB1: track 138.0 -> 348.2 mm, vias 0 -> 1
- net /InputOutputPins/PB5: track 159.0 -> 369.0 mm, vias 0 -> 1
- net /InputOutputPins/PC3: track 94.7 -> 303.2 mm, vias 0 -> 1
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Other:
- board outline added: 149.2 x 215.9 mm
- board text added: "0"
- board text added: "7"
- board text added: "PORT B"
- board text added: "PORT C"
- board text added: "Q0"
- board text added: "Q1"
- board text added: "Q2"
- board text added: "Q3"
- board text added: "Q4"
- board text added: "Q5"
- board text added: "Q6"
- board text added: "Q7"
- board text added: "Q8"
- board text added: "Q9"

Commit message: Rev.1 Upload
Initial completed release
Routing:
- net GND: track 768.8 -> 773.2 mm
- added copper zone on B.Cu, net GND
Other:
- board text added: "AVR_HMI USB CONTROLLED HUMAN-MACHINE-INTERFACE 5V INPUT / OUTPUT"
- board text added: "BOARD CONFIG"
- board text added: "JACOB BOHNERT 000 792 082 MOHAWK COLLEGE"
- board text added: "JLCJLCJLCJLC"
Changed lines of the file:
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@@
   (general
     (thickness 1.6)
-    (drawings 72)
-    (tracks 1409)
+    (drawings 98)
+    (tracks 1415)
     (zones 0)
     (modules 234)
@@
   (layers
     (0 F.Cu signal)
-    (31 B.Cu signal)
+    (31 B.Cu signal hide)
     (32 B.Adhes user)
     (33 F.Adhes user)
@@
     )
   )
+  (gr_text JLCJLCJLCJLC (at 156.21 167.005 -90) (layer F.SilkS)
+    (effects (font (size 1 1) (thickness 0.15)))
+  )
+  (gr_text "AVR_HMI\nUSB CONTROLLED HUMAN-MACHINE-INTERFACE\n5V INPUT / OUTPUT" (at 167.64 156.845 -90) (layer F.SilkS)
+    (effects (font (size 1.524 1.524) (thickness 0.15)))
+  )
+  (gr_line (start 149.86 179.705) (end 149.86 153.67) (layer F.SilkS) (width 0.12))
+  (gr_line (start 161.925 179.705) (end 149.86 179.705) (layer F.SilkS) (width 0.12))
+  (gr_line (start 161.925 153.67) (end 161.925 179.705) (layer F.SilkS) (width 0.12))
+  (gr_line (start 149.86 153.67) (end 161.925 153.67) (layer F.SilkS) (width 0.12))
+  (gr_text "BOARD\nCONFIG" (at 155.575 153.035 -90) (layer F.SilkS)
+    (effects (font (size 3.81 3.81) (thickness 0.15)) (justify right))
+  )
+  (gr_text "JACOB BOHNERT\n000 792 082\nMOHAWK COLLEGE" (at 159.385 212.09) (layer F.Cu)
+    (effects (font (size 1.5 1.5) (thickness 0.3)))
+  )
+  (gr_line (start 136.525 101.6) (end 136.525 107.95) (layer F.SilkS) (width 0.12))
+  (gr_line (start 133.35 104.775) (end 139.7 104.775) (layer F.SilkS) (width 0.12))
+  (gr_circle (center 136.525 104.775) (end 139.7 104.775) (layer F.SilkS) (width 0.12))
+  (gr_line (start 85.725 25.4) (end 85.725 31.75) (layer F.SilkS) (width 0.12))
+  (gr_line (start 82.55 28.575) (end 88.9 28.575) (layer F.SilkS) (width 0.12))
+  (gr_circle (center 85.725 28.575) (end 88.9 28.575) (layer F.SilkS) (width 0.12))
+  (gr_line (start 168.275 219.075) (end 168.275 225.425) (layer F.SilkS) (width 0.12))
+  (gr_line (start 165.1 222.25) (end 171.45 222.25) (layer F.SilkS) (width 0.12))
+  (gr_circle (center 168.275 222.25) (end 171.45 222.25) (layer F.SilkS) (width 0.12))
+  (gr_line (start 168.275 107.95) (end 168.275 114.3) (layer F.SilkS) (width 0.12))
+  (gr_line (start 165.1 111.125) (end 171.45 111.125) (layer F.SilkS) (width 0.12))
+  (gr_circle (center 168.275 111.125) (end 171.45 111.125) (layer F.SilkS) (width 0.12))
+  (gr_line (start 38.1 36.83) (end 38.1 43.18) (layer F.SilkS) (width 0.12))
+  (gr_line (start 34.925 40.005) (end 41.275 40.005) (layer F.SilkS) (width 0.12))
+  (gr_circle (center 38.1 40.005) (end 41.275 40.005) (layer F.SilkS) (width 0.12))
+  (gr_line (start 34.925 222.25) (end 41.275 222.25) (layer F.SilkS) (width 0.12))
+  (gr_line (start 38.1 219.075) (end 38.1 225.425) (layer F.SilkS) (width 0.12))
+  (gr_circle (center 38.1 222.25) (end 41.275 222.25) (layer F.SilkS) (width 0.12))
   (gr_line (start 28.575 234.95) (end 28.575 19.05) (layer Edge.Cuts) (width 0.05))
   (gr_line (start 177.8 234.95) (end 28.575 234.95) (layer Edge.Cuts) (width 0.05))
@@
   (segment (start 42.45 69.37) (end 42.45 67.31) (width 0.25) (layer F.Cu) (net 14))
   (segment (start 39.74 72.08) (end 42.45 69.37) (width 0.25) (layer F.Cu) (net 14))
-  (segment (start 37.990001 32.560001) (end 34.64 29.21) (width 0.25) (layer F.Cu) (net 14))
-  (segment (start 37.990001 58.290001) (end 37.990001 32.560001) (width 0.25) (layer F.Cu) (net 14))
-  (segment (start 39.74 60.04) (end 37.990001 58.290001) (width 0.25) (layer F.Cu) (net 14))
   (segment (start 83.82 73.58) (end 72.39 73.58) (width 0.25) (layer B.Cu) (net 14))
   (segment (start 42.45 68.512081) (end 42.45 67.31) (width 0.25) (layer B.Cu) (net 14))
@@
   (segment (start 39.225001 82.405001) (end 39.225001 92.854999) (width 0.25) (layer B.Cu) (net 14))
   (segment (start 38.1 81.28) (end 39.225001 82.405001) (width 0.25) (layer B.Cu) (net 14))
-  (segment (start 123.19 75.11363) (end 123.19 74.93) (width 0.25) (layer B.Cu) (net 39))
+  (segment (start 38.1 58.4) (end 39.74 60.04) (width 0.25) (layer F.Cu) (net 14))
+  (segment (start 38.1 50.8) (end 38.1 58.4) (width 0.25) (layer F.Cu) (net 14))
+  (segment (start 35.89 29.21) (end 42.545 35.865) (width 0.25) (layer F.Cu) (net 14))
+  (segment (start 34.64 29.21) (end 35.89 29.21) (width 0.25) (layer F.Cu) (net 14))
+  (segment (start 42.545 35.865) (end 42.545 41.91) (width 0.25) (layer F.Cu) (net 14))
+  (segment (start 38.1 46.355) (end 38.1 50.8) (width 0.25) (layer F.Cu) (net 14))
+  (segment (start 42.545 41.91) (end 38.1 46.355) (width 0.25) (layer F.Cu) (net 14))
   (segment (start 40.67 29.18) (end 40.64 29.21) (width 0.25) (layer F.Cu) (net 15))
   (segment (start 40.64 29.21) (end 40.64 31.75) (width 0.25) (layer F.Cu) (net 15))
@@
   (segment (start 123.19 86.01) (end 120.3 86.01) (width 0.25) (layer F.Cu) (net 37))
   (segment (start 90.805 134.62) (end 90.805 130.81) (width 0.25) (layer F.Cu) (net 38))
+  (segment (start 123.19 75.11363) (end 123.19 74.93) (width 0.25) (layer B.Cu) (net 39))
   (via (at 124.46 102.87) (size 0.8) (drill 0.4) (layers F.Cu B.Cu) (net 39))
   (segment (start 139.065 213.995) (end 138.43 213.995) (width 0.25) (layer F.Cu) (net 39))
@@
   (segment (start 107.95 102.87) (end 107.95 105.41) (width 0.25) (layer B.Cu) (net 142))
   (segment (start 86.872588 64.77) (end 93.98 64.77) (width 0.25) (layer F.Cu) (net 143))
-  (segment (start 80.522588 58.42) (end 86.872588 64.77) (width 0.25) (layer F.Cu) (net 143))
-  (segment (start 56.33 58.42) (end 80.522588 58.42) (width 0.25) (layer F.Cu) (net 143))
+  (segment (start 73.025 58.42) (end 79.375 64.77) (width 0.25) (layer F.Cu) (net 143))
   (segment (start 55.245 59.505) (end 56.33 58.42) (width 0.25) (layer F.Cu) (net 143))
   (segment (start 55.245 60.53) (end 55.245 59.505) (width 0.25) (layer F.Cu) (net 143))
+  (segment (start 56.33 58.42) (end 73.025 58.42) (width 0.25) (layer F.Cu) (net 143))
+  (segment (start 79.375 64.77) (end 86.872588 64.77) (width 0.25) (layer F.Cu) (net 143))
   (segment (start 53.975 52.255) (end 58.87 57.15) (width 0.25) (layer F.Cu) (net 144))
   (segment (start 53.975 51.23) (end 53.975 52.255) (width 0.25) (layer F.Cu) (net 144))
   (segment (start 84.968998 62.23) (end 93.98 62.23) (width 0.25) (layer F.Cu) (net 144))
-  (segment (start 79.888998 57.15) (end 84.968998 62.23) (width 0.25) (layer F.Cu) (net 144))
-  (segment (start 58.87 57.15) (end 79.888998 57.15) (width 0.25) (layer F.Cu) (net 144))
+  (segment (start 73.66 57.15) (end 78.74 62.23) (width 0.25) (layer F.Cu) (net 144))
+  (segment (start 58.87 57.15) (end 73.66 57.15) (width 0.25) (layer F.Cu) (net 144))
+  (segment (start 78.74 62.23) (end 85.09 62.23) (width 0.25) (layer F.Cu) (net 144))
   (segment (start 92.71 91.44) (end 99.06 97.79) (width 0.25) (layer F.Cu) (net 145))
   (segment (start 74.542002 91.44) (end 92.71 91.44) (width 0.25) (layer F.Cu) (net 145))
@@
   (segment (start 114.935 221.615) (end 114.935 226.06) (width 0.25) (layer F.Cu) (net 243))
   (segment (start 117.475 226.06) (end 117.475 221.615) (width 0.25) (layer F.Cu) (net 244))
+  (zone (net 14) (net_name GND) (layer B.Cu) (hatch edge 0.508)
+    (connect_pads (clearance 0.508))
+    (min_thickness 0.254)
+    (fill yes (arc_segments 32) (thermal_gap 0.508) (thermal_bridge_width 0.508))
+    (polygon
+      (pts
+        (xy 174.625 232.41) (xy 31.75 231.775) (xy 31.75 22.225) (xy 174.625 22.225)
+      )
+    )
+  )
 )
